File: Sparkdog PF-DI V2/GDI_Control.sch (KiCad schematic (older format))
At the start: 8 parts, among them U900 SN74AHCT02, U901 SN74AHCT02, U902 SN74AHCT08, U903 SN74AHCT08

Commit message: Commit schematic changes, new parts library footprints and step files, PCB design file.
Parts:
- CD900, CD901, CD902, CD903: footprint (none) -> Samacsys:RESC1608X55N
- U900, U901, U902, U903: footprint (none) -> Samacsys:SOP65P640X110-14N
Changed lines of the file:
@@
 F 0 "U902" H 7600 3315 50  0000 C CNN
 F 1 "SN74AHCT08" H 7600 3224 50  0000 C CNN
-F 2 "" H 7400 2350 50  0001 C CNN
+F 2 "Samacsys:SOP65P640X110-14N" H 7400 2350 50  0001 C CNN
 F 3 "" H 7400 2350 50  0001 C CNN
 	1    7400 2350
@@
 F 0 "U900" H 6100 3665 50  0000 C CNN
 F 1 "SN74AHCT02" H 6100 3574 50  0000 C CNN
-F 2 "" H 5900 2700 50  0001 C CNN
+F 2 "Samacsys:SOP65P640X110-14N" H 5900 2700 50  0001 C CNN
 F 3 "" H 5900 2700 50  0001 C CNN
 	1    5900 2700
@@
 F 0 "CD900" H 4365 1746 50  0000 L CNN
 F 1 "0603 100nF" H 4365 1655 50  0000 L CNN
-F 2 "" H 4288 1550 50  0001 C CNN
+F 2 "Samacsys:RESC1608X55N" H 4288 1550 50  0001 C CNN
 F 3 "~" H 4250 1700 50  0001 C CNN
 	1    4250 1700
@@
 F 0 "CD901" H 5065 1746 50  0000 L CNN
 F 1 "0603 100nF" H 5065 1655 50  0000 L CNN
-F 2 "" H 4988 1550 50  0001 C CNN
+F 2 "Samacsys:RESC1608X55N" H 4988 1550 50  0001 C CNN
 F 3 "~" H 4950 1700 50  0001 C CNN
 	1    4950 1700
@@
 F 0 "U903" H 7600 5815 50  0000 C CNN
 F 1 "SN74AHCT08" H 7600 5724 50  0000 C CNN
-F 2 "" H 7400 4850 50  0001 C CNN
+F 2 "Samacsys:SOP65P640X110-14N" H 7400 4850 50  0001 C CNN
 F 3 "" H 7400 4850 50  0001 C CNN
 	1    7400 4850
@@
 F 0 "U901" H 6100 6165 50  0000 C CNN
 F 1 "SN74AHCT02" H 6100 6074 50  0000 C CNN
-F 2 "" H 5900 5200 50  0001 C CNN
+F 2 "Samacsys:SOP65P640X110-14N" H 5900 5200 50  0001 C CNN
 F 3 "" H 5900 5200 50  0001 C CNN
 	1    5900 5200
@@
 F 0 "CD902" H 4365 4246 50  0000 L CNN
 F 1 "0603 100nF" H 4365 4155 50  0000 L CNN
-F 2 "" H 4288 4050 50  0001 C CNN
+F 2 "Samacsys:RESC1608X55N" H 4288 4050 50  0001 C CNN
 F 3 "~" H 4250 4200 50  0001 C CNN
 	1    4250 4200
@@
 F 0 "CD903" H 5065 4246 50  0000 L CNN
 F 1 "0603 100nF" H 5065 4155 50  0000 L CNN
-F 2 "" H 4988 4050 50  0001 C CNN
+F 2 "Samacsys:RESC1608X55N" H 4988 4050 50  0001 C CNN
 F 3 "~" H 4950 4200 50  0001 C CNN
 	1    4950 4200
