File: Sparkdog PF-DI V2/Knock.sch (KiCad schematic (older format))
At the start: 23 parts, among them U400 AD8620, U401 AD8620

Commit message: Commit schematic changes, new parts library footprints and step files, PCB design file.
Parts:
- C400, C401, CD400, CD401: value 100nF -> 0603 100nF; footprint (none) -> Samacsys:RESC1608X55N
- C402, C403, C404, C405: value 1nF -> 0603 1nF; footprint (none) -> Samacsys:RESC1608X55N
- R400, R401: value 4.7k -> 0603 4.7k; footprint (none) -> Samacsys:RESC1608X55N
- R402, R403, R406, R407, R408, R409: footprint (none) -> Samacsys:RESC1608X55N
- R404, R405: value 47k -> 0603 47k; footprint (none) -> Samacsys:RESC1608X55N
- RN400, RN401, RN402: footprint (none) -> Samacsys:742C083103JP
- U400, U401: value AD8620 -> TLV9052; footprint (none) -> Samacsys:SOT65P280X110-8N
Changed lines of the file:
@@
 P 5100 1750
 F 0 "U400" H 5100 2117 50  0000 C CNN
-F 1 "AD8620" H 5100 2026 50  0000 C CNN
-F 2 "" H 5100 1750 50  0001 C CNN
+F 1 "TLV9052" H 5100 2026 50  0000 C CNN
+F 2 "Samacsys:SOT65P280X110-8N" H 5100 1750 50  0001 C CNN
 F 3 "https://www.analog.com/media/en/technical-documentation/data-sheets/AD8610_8620.pdf" H 5100 1750 50  0001 C CNN
 	1    5100 1750
@@
 P 5250 2500
 F 0 "U400" H 5250 2867 50  0000 C CNN
-F 1 "AD8620" H 5250 2776 50  0000 C CNN
-F 2 "" H 5250 2500 50  0001 C CNN
+F 1 "TLV9052" H 5250 2776 50  0000 C CNN
+F 2 "Samacsys:SOT65P280X110-8N" H 5250 2500 50  0001 C CNN
 F 3 "https://www.analog.com/media/en/technical-documentation/data-sheets/AD8610_8620.pdf" H 5250 2500 50  0001 C CNN
 	2    5250 2500
@@
 P 6350 2050
 F 0 "U400" H 6308 2096 50  0000 L CNN
-F 1 "AD8620" H 6308 2005 50  0000 L CNN
-F 2 "" H 6350 2050 50  0001 C CNN
+F 1 "TLV9052" H 6308 2005 50  0000 L CNN
+F 2 "Samacsys:SOT65P280X110-8N" H 6350 2050 50  0001 C CNN
 F 3 "https://www.analog.com/media/en/technical-documentation/data-sheets/AD8610_8620.pdf" H 6350 2050 50  0001 C CNN
 	3    6350 2050
@@
 F 0 "RN400" V 2183 3150 50  0000 C CNN
 F 1 "220k" V 2274 3150 50  0000 C CNN
-F 2 "" V 2875 3150 50  0001 C CNN
+F 2 "Samacsys:742C083103JP" V 2875 3150 50  0001 C CNN
 F 3 "~" H 2600 3150 50  0001 C CNN
 	1    2600 3150
@@
 F 0 "RN401" V 3483 3150 50  0000 C CNN
 F 1 "220R" V 3574 3150 50  0000 C CNN
-F 2 "" V 4175 3150 50  0001 C CNN
+F 2 "Samacsys:742C083103JP" V 4175 3150 50  0001 C CNN
 F 3 "~" H 3900 3150 50  0001 C CNN
 	1    3900 3150
@@
 F 0 "RN402" V 4133 3150 50  0000 C CNN
 F 1 "220k" V 4224 3150 50  0000 C CNN
-F 2 "" V 4825 3150 50  0001 C CNN
+F 2 "Samacsys:742C083103JP" V 4825 3150 50  0001 C CNN
 F 3 "~" H 4550 3150 50  0001 C CNN
 	1    4550 3150
@@
 P 5400 3900
 F 0 "U401" H 5400 4267 50  0000 C CNN
-F 1 "AD8620" H 5400 4176 50  0000 C CNN
-F 2 "" H 5400 3900 50  0001 C CNN
+F 1 "TLV9052" H 5400 4176 50  0000 C CNN
+F 2 "Samacsys:SOT65P280X110-8N" H 5400 3900 50  0001 C CNN
 F 3 "https://www.analog.com/media/en/technical-documentation/data-sheets/AD8610_8620.pdf" H 5400 3900 50  0001 C CNN
 	1    5400 3900
@@
 P 5400 4750
 F 0 "U401" H 5400 5117 50  0000 C CNN
-F 1 "AD8620" H 5400 5026 50  0000 C CNN
-F 2 "" H 5400 4750 50  0001 C CNN
+F 1 "TLV9052" H 5400 5026 50  0000 C CNN
+F 2 "Samacsys:SOT65P280X110-8N" H 5400 4750 50  0001 C CNN
 F 3 "https://www.analog.com/media/en/technical-documentation/data-sheets/AD8610_8620.pdf" H 5400 4750 50  0001 C CNN
 	2    5400 4750
@@
 P 6350 4200
 F 0 "U401" H 6308 4246 50  0000 L CNN
-F 1 "AD8620" H 6308 4155 50  0000 L CNN
-F 2 "" H 6350 4200 50  0001 C CNN
+F 1 "TLV9052" H 6308 4155 50  0000 L CNN
+F 2 "Samacsys:SOT65P280X110-8N" H 6350 4200 50  0001 C CNN
 F 3 "https://www.analog.com/media/en/technical-documentation/data-sheets/AD8610_8620.pdf" H 6350 4200 50  0001 C CNN
 	3    6350 4200
@@
 P 2700 2450
 F 0 "R400" V 2493 2450 50  0000 C CNN
-F 1 "4.7k" V 2584 2450 50  0000 C CNN
-F 2 "" V 2630 2450 50  0001 C CNN
+F 1 "0603 4.7k" V 2584 2450 50  0000 C CNN
+F 2 "Samacsys:RESC1608X55N" V 2630 2450 50  0001 C CNN
 F 3 "~" H 2700 2450 50  0001 C CNN
 	1    2700 2450
@@
 P 2700 3800
 F 0 "R401" V 2493 3800 50  0000 C CNN
-F 1 "4.7k" V 2584 3800 50  0000 C CNN
-F 2 "" V 2630 3800 50  0001 C CNN
+F 1 "0603 4.7k" V 2584 3800 50  0000 C CNN
+F 2 "Samacsys:RESC1608X55N" V 2630 3800 50  0001 C CNN
 F 3 "~" H 2700 3800 50  0001 C CNN
 	1    2700 3800
@@
 P 3900 3800
 F 0 "R405" V 3693 3800 50  0000 C CNN
-F 1 "47k" V 3784 3800 50  0000 C CNN
-F 2 "" V 3830 3800 50  0001 C CNN
+F 1 "0603 47k" V 3784 3800 50  0000 C CNN
+F 2 "Samacsys:RESC1608X55N" V 3830 3800 50  0001 C CNN
 F 3 "~" H 3900 3800 50  0001 C CNN
 	1    3900 3800
@@
 F 0 "R403" V 3293 4050 50  0000 C CNN
 F 1 "0603 47k" V 3384 4050 50  0000 C CNN
-F 2 "" V 3430 4050 50  0001 C CNN
+F 2 "Samacsys:RESC1608X55N" V 3430 4050 50  0001 C CNN
 F 3 "~" H 3500 4050 50  0001 C CNN
 	1    3500 4050
@@
 P 3900 2450
 F 0 "R404" V 3693 2450 50  0000 C CNN
-F 1 "47k" V 3784 2450 50  0000 C CNN
-F 2 "" V 3830 2450 50  0001 C CNN
+F 1 "0603 47k" V 3784 2450 50  0000 C CNN
+F 2 "Samacsys:RESC1608X55N" V 3830 2450 50  0001 C CNN
 F 3 "~" H 3900 2450 50  0001 C CNN
 	1    3900 2450
@@
 F 0 "R402" V 3293 2150 50  0000 C CNN
 F 1 "0603 47k" V 3384 2150 50  0000 C CNN
-F 2 "" V 3430 2150 50  0001 C CNN
+F 2 "Samacsys:RESC1608X55N" V 3430 2150 50  0001 C CNN
 F 3 "~" H 3500 2150 50  0001 C CNN
 	1    3500 2150
@@
 P 3150 2450
 F 0 "C402" V 2898 2450 50  0000 C CNN
-F 1 "1nF" V 2989 2450 50  0000 C CNN
-F 2 "" H 3188 2300 50  0001 C CNN
+F 1 "0603 1nF" V 2989 2450 50  0000 C CNN
+F 2 "Samacsys:RESC1608X55N" H 3188 2300 50  0001 C CNN
 F 3 "~" H 3150 2450 50  0001 C CNN
 	1    3150 2450
@@
 P 1950 2700
 F 0 "C400" H 2065 2746 50  0000 L CNN
-F 1 "100nF" H 2065 2655 50  0000 L CNN
-F 2 "" H 1988 2550 50  0001 C CNN
+F 1 "0603 100nF" H 2065 2655 50  0000 L CNN
+F 2 "Samacsys:RESC1608X55N" H 1988 2550 50  0001 C CNN
 F 3 "~" H 1950 2700 50  0001 C CNN
 	1    1950 2700
@@
 P 1950 3750
 F 0 "C401" H 2065 3796 50  0000 L CNN
-F 1 "100nF" H 2065 3705 50  0000 L CNN
-F 2 "" H 1988 3600 50  0001 C CNN
+F 1 "0603 100nF" H 2065 3705 50  0000 L CNN
+F 2 "Samacsys:RESC1608X55N" H 1988 3600 50  0001 C CNN
 F 3 "~" H 1950 3750 50  0001 C CNN
 	1    1950 3750
@@
 P 6700 2050
 F 0 "CD400" H 6815 2096 50  0000 L CNN
-F 1 "100nF" H 6815 2005 50  0000 L CNN
-F 2 "" H 6738 1900 50  0001 C CNN
+F 1 "0603 100nF" H 6815 2005 50  0000 L CNN
+F 2 "Samacsys:RESC1608X55N" H 6738 1900 50  0001 C CNN
 F 3 "~" H 6700 2050 50  0001 C CNN
 	1    6700 2050
@@
 P 6700 4200
 F 0 "CD401" H 6815 4246 50  0000 L CNN
-F 1 "100nF" H 6815 4155 50  0000 L CNN
-F 2 "" H 6738 4050 50  0001 C CNN
+F 1 "0603 100nF" H 6815 4155 50  0000 L CNN
+F 2 "Samacsys:RESC1608X55N" H 6738 4050 50  0001 C CNN
 F 3 "~" H 6700 4200 50  0001 C CNN
 	1    6700 4200
@@
 P 4800 2250
 F 0 "C404" H 4915 2296 50  0000 L CNN
-F 1 "1nF" H 4915 2205 50  0000 L CNN
-F 2 "" H 4838 2100 50  0001 C CNN
+F 1 "0603 1nF" H 4915 2205 50  0000 L CNN
+F 2 "Samacsys:RESC1608X55N" H 4838 2100 50  0001 C CNN
 F 3 "~" H 4800 2250 50  0001 C CNN
 	1    4800 2250
@@
 P 4500 4500
 F 0 "C405" H 4615 4546 50  0000 L CNN
-F 1 "1nF" H 4615 4455 50  0000 L CNN
-F 2 "" H 4538 4350 50  0001 C CNN
+F 1 "0603 1nF" H 4615 4455 50  0000 L CNN
+F 2 "Samacsys:RESC1608X55N" H 4538 4350 50  0001 C CNN
 F 3 "~" H 4500 4500 50  0001 C CNN
 	1    4500 4500
@@
 P 3150 3800
 F 0 "C403" V 2898 3800 50  0000 C CNN
-F 1 "1nF" V 2989 3800 50  0000 C CNN
-F 2 "" H 3188 3650 50  0001 C CNN
+F 1 "0603 1nF" V 2989 3800 50  0000 C CNN
+F 2 "Samacsys:RESC1608X55N" H 3188 3650 50  0001 C CNN
 F 3 "~" H 3150 3800 50  0001 C CNN
 	1    3150 3800
@@
 F 0 "R408" V 1393 2550 50  0000 C CNN
 F 1 "0603 1k" V 1484 2550 50  0000 C CNN
-F 2 "" V 1530 2550 50  0001 C CNN
+F 2 "Samacsys:RESC1608X55N" V 1530 2550 50  0001 C CNN
 F 3 "~" H 1600 2550 50  0001 C CNN
 	1    1600 2550
@@
 F 0 "R409" V 1393 3900 50  0000 C CNN
 F 1 "0603 1k" V 1484 3900 50  0000 C CNN
-F 2 "" V 1530 3900 50  0001 C CNN
+F 2 "Samacsys:RESC1608X55N" V 1530 3900 50  0001 C CNN
 F 3 "~" H 1600 3900 50  0001 C CNN
 	1    1600 3900
@@
 F 0 "R406" V 5593 2800 50  0000 C CNN
 F 1 "0603 1k" V 5684 2800 50  0000 C CNN
-F 2 "" V 5730 2800 50  0001 C CNN
+F 2 "Samacsys:RESC1608X55N" V 5730 2800 50  0001 C CNN
 F 3 "~" H 5800 2800 50  0001 C CNN
 	1    5800 2800
@@
 F 0 "R407" V 5743 5050 50  0000 C CNN
 F 1 "0603 1k" V 5834 5050 50  0000 C CNN
-F 2 "" V 5880 5050 50  0001 C CNN
+F 2 "Samacsys:RESC1608X55N" V 5880 5050 50  0001 C CNN
 F 3 "~" H 5950 5050 50  0001 C CNN
 	1    5950 5050
