File: Sparkdog PF-DI V2/VVT.sch (KiCad schematic (older format))
At the start: 23 parts, among them U200 IRF7907TRPBF, U201 Dual_Trans_Array_NPN, U202 Dual_Trans_Array_NPN, U203 Dual_Trans_Array_PNP, U204 Dual_Trans_Array_PNP, U205 74AHC14PW,118

Commit message: Commit schematic changes, new parts library footprints and step files, PCB design file.
Parts:
- C200, C201, C202, C203: value C -> 0603 1nF; footprint (none) -> Samacsys:RESC1608X55N
- CD200: footprint (none) -> Samacsys:RESC1608X55N
- D200, D201, D202, D203: footprint SOT96P237X111-3N -> Samacsys:SOT96P237X111-3N
- R200, R201: value 1210 0.1R -> 1206 0.1R; footprint (none) -> Samacsys:RESC3216X60N
- RN200, RN201, RN202, RN203, RN204, RN205: footprint (none) -> Samacsys:742C083103JP
- U200: footprint SOIC127P600X175-8N -> Samacsys:SOIC127P600X175-8N
- U201, U202, U203, U204: footprint (none) -> Sparkdog PF-DI V2:SOT-363-6
- U205: footprint SOP65P640X110-14N -> Samacsys:SOP65P640X110-14N
Changed lines of the file:
@@
 F 0 "U205" H 7050 4415 50  0000 C CNN
 F 1 "74AHC14PW,118" H 7050 4324 50  0000 C CNN
-F 2 "SOP65P640X110-14N" H 7400 4250 50  0001 L CNN
+F 2 "Samacsys:SOP65P640X110-14N" H 7400 4250 50  0001 L CNN
 F 3 "https://componentsearchengine.com/Datasheets/1/74AHC14PW,118.pdf" H 7400 4150 50  0001 L CNN
 F 4 "74AHC(T)14 - Hex inverting Schmitt trigger@en-us" H 7400 4050 50  0001 L CNN "Description"
@@
 F 0 "U201" H 6325 2075 50  0000 C CNN
 F 1 "Dual_Trans_Array_NPN" H 6325 1984 50  0000 C CNN
-F 2 "" H 6150 1600 50  0001 C CNN
+F 2 "Sparkdog PF-DI V2:SOT-363-6" H 6150 1600 50  0001 C CNN
 F 3 "" H 6150 1600 50  0001 C CNN
 	1    6150 1600
@@
 F 0 "U202" H 7925 2075 50  0000 C CNN
 F 1 "Dual_Trans_Array_NPN" H 7925 1984 50  0000 C CNN
-F 2 "" H 7750 1600 50  0001 C CNN
+F 2 "Sparkdog PF-DI V2:SOT-363-6" H 7750 1600 50  0001 C CNN
 F 3 "" H 7750 1600 50  0001 C CNN
 	1    7750 1600
@@
 F 0 "RN201" V 5333 4150 50  0000 C CNN
 F 1 "1206 10k" V 5424 4150 50  0000 C CNN
-F 2 "" V 6025 4150 50  0001 C CNN
+F 2 "Samacsys:742C083103JP" V 6025 4150 50  0001 C CNN
 F 3 "~" H 5750 4150 50  0001 C CNN
 	1    5750 4150
@@
 F 0 "RN202" V 5333 4900 50  0000 C CNN
 F 1 "1206 10k" V 5424 4900 50  0000 C CNN
-F 2 "" V 6025 4900 50  0001 C CNN
+F 2 "Samacsys:742C083103JP" V 6025 4900 50  0001 C CNN
 F 3 "~" H 5750 4900 50  0001 C CNN
 	1    5750 4900
@@
 F 0 "RN205" V 8183 4850 50  0000 C CNN
 F 1 "1206 10k" V 8274 4850 50  0000 C CNN
-F 2 "" V 8875 4850 50  0001 C CNN
+F 2 "Samacsys:742C083103JP" V 8875 4850 50  0001 C CNN
 F 3 "~" H 8600 4850 50  0001 C CNN
 	1    8600 4850
@@
 F 0 "RN204" V 8183 4200 50  0000 C CNN
 F 1 "1206 10k" V 8274 4200 50  0000 C CNN
-F 2 "" V 8875 4200 50  0001 C CNN
+F 2 "Samacsys:742C083103JP" V 8875 4200 50  0001 C CNN
 F 3 "~" H 8600 4200 50  0001 C CNN
 	1    8600 4200
@@
 F 0 "D200" H 7950 3335 50  0000 C CNN
 F 1 "BZX84C5V1LT1G" H 7950 3426 50  0000 C CNN
-F 2 "SOT96P237X111-3N" H 8250 3800 50  0001 L CNN
+F 2 "Samacsys:SOT96P237X111-3N" H 8250 3800 50  0001 L CNN
 F 3 "http://www.onsemi.com/pub/Collateral/BZX84C2V4LT1-D.PDF" H 8250 3700 50  0001 L CNN
 F 4 "250 mW 5.1 V +/-5% Zener Diode Voltage Regulator" H 8250 3600 50  0001 L CNN "Description"
@@
 F 0 "D201" H 7950 4985 50  0000 C CNN
 F 1 "BZX84C5V1LT1G" H 7950 5076 50  0000 C CNN
-F 2 "SOT96P237X111-3N" H 8250 5450 50  0001 L CNN
+F 2 "Samacsys:SOT96P237X111-3N" H 8250 5450 50  0001 L CNN
 F 3 "http://www.onsemi.com/pub/Collateral/BZX84C2V4LT1-D.PDF" H 8250 5350 50  0001 L CNN
 F 4 "250 mW 5.1 V +/-5% Zener Diode Voltage Regulator" H 8250 5250 50  0001 L CNN "Description"
@@
 F 0 "D202" H 8772 3554 50  0000 R CNN
 F 1 "BZX84C5V1LT1G" H 8772 3645 50  0000 R CNN
-F 2 "SOT96P237X111-3N" H 9750 3700 50  0001 L CNN
+F 2 "Samacsys:SOT96P237X111-3N" H 9750 3700 50  0001 L CNN
 F 3 "http://www.onsemi.com/pub/Collateral/BZX84C2V4LT1-D.PDF" H 9750 3600 50  0001 L CNN
 F 4 "250 mW 5.1 V +/-5% Zener Diode Voltage Regulator" H 9750 3500 50  0001 L CNN "Description"
@@
 F 0 "D203" H 9450 5185 50  0000 C CNN
 F 1 "BZX84C5V1LT1G" H 9450 5276 50  0000 C CNN
-F 2 "SOT96P237X111-3N" H 9750 5650 50  0001 L CNN
+F 2 "Samacsys:SOT96P237X111-3N" H 9750 5650 50  0001 L CNN
 F 3 "http://www.onsemi.com/pub/Collateral/BZX84C2V4LT1-D.PDF" H 9750 5550 50  0001 L CNN
 F 4 "250 mW 5.1 V +/-5% Zener Diode Voltage Regulator" H 9750 5450 50  0001 L CNN "Description"
@@
 P 6350 3550
 F 0 "C200" H 6465 3596 50  0000 L CNN
-F 1 "C" H 6465 3505 50  0000 L CNN
-F 2 "" H 6388 3400 50  0001 C CNN
+F 1 "0603 1nF" H 6465 3505 50  0000 L CNN
+F 2 "Samacsys:RESC1608X55N" H 6388 3400 50  0001 C CNN
 F 3 "~" H 6350 3550 50  0001 C CNN
 	1    6350 3550
@@
 P 7900 3450
 F 0 "C202" H 8015 3496 50  0000 L CNN
-F 1 "C" H 8015 3405 50  0000 L CNN
-F 2 "" H 7938 3300 50  0001 C CNN
+F 1 "0603 1nF" H 8015 3405 50  0000 L CNN
+F 2 "Samacsys:RESC1608X55N" H 7938 3300 50  0001 C CNN
 F 3 "~" H 7900 3450 50  0001 C CNN
 	1    7900 3450
@@
 P 7900 5700
 F 0 "C203" H 8015 5746 50  0000 L CNN
-F 1 "C" H 8015 5655 50  0000 L CNN
-F 2 "" H 7938 5550 50  0001 C CNN
+F 1 "0603 1nF" H 8015 5655 50  0000 L CNN
+F 2 "Samacsys:RESC1608X55N" H 7938 5550 50  0001 C CNN
 F 3 "~" H 7900 5700 50  0001 C CNN
 	1    7900 5700
@@
 P 6150 5500
 F 0 "C201" H 6265 5546 50  0000 L CNN
-F 1 "C" H 6265 5455 50  0000 L CNN
-F 2 "" H 6188 5350 50  0001 C CNN
+F 1 "0603 1nF" H 6265 5455 50  0000 L CNN
+F 2 "Samacsys:RESC1608X55N" H 6188 5350 50  0001 C CNN
 F 3 "~" H 6150 5500 50  0001 C CNN
 	1    6150 5500
@@
 F 0 "CD200" H 7165 6196 50  0000 L CNN
 F 1 "0603 100nF" H 7165 6105 50  0000 L CNN
-F 2 "" H 7088 6000 50  0001 C CNN
+F 2 "Samacsys:RESC1608X55N" H 7088 6000 50  0001 C CNN
 F 3 "~" H 7050 6150 50  0001 C CNN
 	1    7050 6150
@@
 F 0 "U203" H 6325 2725 50  0000 C CNN
 F 1 "Dual_Trans_Array_PNP" H 6325 2634 50  0000 C CNN
-F 2 "" H 6150 2250 50  0001 C CNN
+F 2 "Sparkdog PF-DI V2:SOT-363-6" H 6150 2250 50  0001 C CNN
 F 3 "" H 6150 2250 50  0001 C CNN
 	1    6150 2250
@@
 F 0 "U204" H 7925 2725 50  0000 C CNN
 F 1 "Dual_Trans_Array_PNP" H 7925 2634 50  0000 C CNN
-F 2 "" H 7750 2250 50  0001 C CNN
+F 2 "Sparkdog PF-DI V2:SOT-363-6" H 7750 2250 50  0001 C CNN
 F 3 "" H 7750 2250 50  0001 C CNN
 	1    7750 2250
@@
 F 0 "RN203" H 7538 2896 50  0000 L CNN
 F 1 "1206 470R" H 7538 2805 50  0000 L CNN
-F 2 "" V 7625 2850 50  0001 C CNN
+F 2 "Samacsys:742C083103JP" V 7625 2850 50  0001 C CNN
 F 3 "~" H 7350 2850 50  0001 C CNN
 	1    7350 2850
@@
 F 0 "U200" H 3500 2765 50  0000 C CNN
 F 1 "IRF7907TRPBF" H 3500 2674 50  0000 C CNN
-F 2 "SOIC127P600X175-8N" H 3850 2600 50  0001 L CNN
+F 2 "Samacsys:SOIC127P600X175-8N" H 3850 2600 50  0001 L CNN
 F 3 "https://www.infineon.com/dgdl/irf7907pbf.pdf?fileId=5546d462533600a40153560c992e1d39" H 3850 2500 50  0001 L CNN
 F 4 "IRF7907TRPBF Dual N-Channel MOSFET, 9.1 A, 11 A, 30 V HEXFET, 8-Pin SOIC Infineon" H 3850 2400 50  0001 L CNN "Description"
@@
 F 0 "RN200" V 1833 2700 50  0000 C CNN
 F 1 "1206 10k" V 1924 2700 50  0000 C CNN
-F 2 "" V 2525 2700 50  0001 C CNN
+F 2 "Samacsys:742C083103JP" V 2525 2700 50  0001 C CNN
 F 3 "~" H 2250 2700 50  0001 C CNN
 	1    2250 2700
@@
 P 2800 2200
 F 0 "R200" H 2870 2246 50  0000 L CNN
-F 1 "1210 0.1R" H 2870 2155 50  0000 L CNN
-F 2 "" V 2730 2200 50  0001 C CNN
+F 1 "1206 0.1R" H 2870 2155 50  0000 L CNN
+F 2 "Samacsys:RESC3216X60N" V 2730 2200 50  0001 C CNN
 F 3 "~" H 2800 2200 50  0001 C CNN
 	1    2800 2200
@@
 P 2800 3100
 F 0 "R201" H 2870 3146 50  0000 L CNN
-F 1 "1210 0.1R" H 2870 3055 50  0000 L CNN
-F 2 "" V 2730 3100 50  0001 C CNN
+F 1 "1206 0.1R" H 2870 3055 50  0000 L CNN
+F 2 "Samacsys:RESC3216X60N" V 2730 3100 50  0001 C CNN
 F 3 "~" H 2800 3100 50  0001 C CNN
 	1    2800 3100
