File: Sparkdog PF-DI V2/_autosave-ETC PROCESSOR.sch (KiCad schematic (older format))
At the start: 21 parts, among them J600 M50-3610542R, U600 MK10DX128VLK7, U601 TLV809EA29DCKR, X600 Crystal

Commit message: Commit schematic changes, new parts library footprints and step files, PCB design file.
Parts:
- C600, C601, CD600, CD601, CD602, CD603, CD604, CD605, CD606, R600: footprint Samacsys:RESC1608X55N -> (none)
- J600: footprint Samacsys:M503610542 -> M503610542
- RN600, RN601, RN602, RN603, RN604, RN605: footprint Samacsys:742C083103JP -> (none)
- RN605: renamed from RN606; footprint Samacsys:742C083103JP -> (none)
- U600: footprint Sparkdog PF-DI V2:MK10DX128VLK7 -> (none)
- U601: footprint Samacsys:SOT65P210X110-3N -> SOT65P210X110-3N
- X600: footprint Samacsys:ECS49205PXTR -> (none)
Other:
- note added: "ETC PROCESSOR - can be used as an alternate low cost processor with Teensy not fitted."
Changed lines of the file:
@@
 F 0 "J600" V 4950 5100 50  0000 L CNN
 F 1 "M50-3610542R" V 5050 5100 50  0000 L CNN
-F 2 "Samacsys:M503610542" H 5300 6450 50  0001 L CNN
+F 2 "M503610542" H 5300 6450 50  0001 L CNN
 F 3 "https://cdn.harwin.com/pdfs/M50-361.pdf" H 5300 6350 50  0001 L CNN
 F 4 "HARWIN - M50-3610542R - CONNECTOR, HEADER, 10POS, 2ROW, 1.27MM" H 5300 6250 50  0001 L CNN "Description"
@@
 F 0 "C601" V 8200 5750 50  0000 C CNN
 F 1 "0603 10pF" V 8250 6100 50  0000 C CNN
-F 2 "Samacsys:RESC1608X55N" H 8038 5700 50  0001 C CNN
+F 2 "" H 8038 5700 50  0001 C CNN
 F 3 "~" H 8000 5850 50  0001 C CNN
 	1    8000 5850
@@
 F 0 "C600" V 7550 5300 50  0000 C CNN
 F 1 "0603 10pF" V 7650 5450 50  0000 C CNN
-F 2 "Samacsys:RESC1608X55N" H 8038 5300 50  0001 C CNN
+F 2 "" H 8038 5300 50  0001 C CNN
 F 3 "~" H 8000 5450 50  0001 C CNN
 	1    8000 5450
@@
 F 0 "X600" V 7304 5781 50  0000 L CNN
 F 1 "Crystal" V 7395 5781 50  0000 L CNN
-F 2 "Samacsys:ECS49205PXTR" H 7350 5650 50  0001 C CNN
+F 2 "" H 7350 5650 50  0001 C CNN
 F 3 "~" H 7350 5650 50  0001 C CNN
 	1    7350 5650
@@
 F 0 "CD606" H 10515 5446 50  0000 L CNN
 F 1 "0603 100nF" H 10515 5355 50  0000 L CNN
-F 2 "Samacsys:RESC1608X55N" H 10438 5250 50  0001 C CNN
+F 2 "" H 10438 5250 50  0001 C CNN
 F 3 "~" H 10400 5400 50  0001 C CNN
 	1    10400 5400
@@
 F 0 "R600" V 8243 5250 50  0000 C CNN
 F 1 "0603 1k" V 8334 5250 50  0000 C CNN
-F 2 "Samacsys:RESC1608X55N" V 8380 5250 50  0001 C CNN
+F 2 "" V 8380 5250 50  0001 C CNN
 F 3 "~" H 8450 5250 50  0001 C CNN
 	1    8450 5250
@@
 F 0 "U601" H 9650 5415 50  0000 C CNN
 F 1 "TLV809EA29DCKR" H 9650 5324 50  0000 C CNN
-F 2 "Samacsys:SOT65P210X110-3N" H 10100 5250 50  0001 L CNN
+F 2 "SOT65P210X110-3N" H 10100 5250 50  0001 L CNN
 F 3 "https://www.ti.com/lit/ds/symlink/tlv809e.pdf?ts=1605772627929&ref_url=https%253A%252F%252Fwww.ti.com%252Fsitesearch%252Fdocs%252Funiversalsearch.tsp%253FsearchTerm%253DTLV809EA29DCKR" H 10100 5150 50  0001 L CNN
 F 4 "Supervisory Circuits Low-power 3-pin voltage supervisor (reset IC) with active-low, push-pull reset 3-SC70 -40 to 125" H 10100 5050 50  0001 L CNN "Description"
@@
 F 0 "RN604" H 6438 6696 50  0000 L CNN
 F 1 "1206 1k" H 6438 6605 50  0000 L CNN
-F 2 "Samacsys:742C083103JP" V 6525 6650 50  0001 C CNN
+F 2 "" V 6525 6650 50  0001 C CNN
 F 3 "~" H 6250 6650 50  0001 C CNN
 	1    6250 6650
@@
 F 0 "RN605" H 6238 1246 50  0000 L CNN
 F 1 "1206 10k" H 6238 1155 50  0000 L CNN
-F 2 "Samacsys:742C083103JP" V 6325 1200 50  0001 C CNN
+F 2 "" V 6325 1200 50  0001 C CNN
 F 3 "~" H 6050 1200 50  0001 C CNN
 	1    6050 1200
@@
 F 0 "RN600" V 2183 3650 50  0000 C CNN
 F 1 "1206 10k" V 2274 3650 50  0000 C CNN
-F 2 "Samacsys:742C083103JP" V 2875 3650 50  0001 C CNN
+F 2 "" V 2875 3650 50  0001 C CNN
 F 3 "~" H 2600 3650 50  0001 C CNN
 	1    2600 3650
@@
 F 0 "RN601" V 2850 4750 50  0000 C CNN
 F 1 "1206 100k" V 2950 4850 50  0000 C CNN
-F 2 "Samacsys:742C083103JP" V 2875 4850 50  0001 C CNN
+F 2 "" V 2875 4850 50  0001 C CNN
 F 3 "~" H 2600 4850 50  0001 C CNN
 	1    2600 4850
@@
 F 0 "RN602" H 4600 2750 50  0000 L CNN
 F 1 "1206 10k" H 4600 2650 50  0000 L CNN
-F 2 "Samacsys:742C083103JP" V 5525 2500 50  0001 C CNN
+F 2 "" V 5525 2500 50  0001 C CNN
 F 3 "~" H 5250 2500 50  0001 C CNN
 	1    5250 2500
@@
 F 0 "RN603" H 6638 2546 50  0000 L CNN
 F 1 "1206 10k" H 6638 2455 50  0000 L CNN
-F 2 "Samacsys:742C083103JP" V 6725 2500 50  0001 C CNN
+F 2 "" V 6725 2500 50  0001 C CNN
 F 3 "~" H 6450 2500 50  0001 C CNN
 	1    6450 2500
@@
 F 0 "CD603" H 3765 5246 50  0000 L CNN
 F 1 "0603 100nF" H 3765 5155 50  0000 L CNN
-F 2 "Samacsys:RESC1608X55N" H 3688 5050 50  0001 C CNN
+F 2 "" H 3688 5050 50  0001 C CNN
 F 3 "~" H 3650 5200 50  0001 C CNN
 	1    3650 5200
@@
 F 0 "CD605" H 7365 6296 50  0000 L CNN
 F 1 "0603 100nF" H 7365 6205 50  0000 L CNN
-F 2 "Samacsys:RESC1608X55N" H 7288 6100 50  0001 C CNN
+F 2 "" H 7288 6100 50  0001 C CNN
 F 3 "~" H 7250 6250 50  0001 C CNN
 	1    7250 6250
@@
 F 0 "CD601" H 3615 2696 50  0000 L CNN
 F 1 "0603 100nF" H 3615 2605 50  0000 L CNN
-F 2 "Samacsys:RESC1608X55N" H 3538 2500 50  0001 C CNN
+F 2 "" H 3538 2500 50  0001 C CNN
 F 3 "~" H 3500 2650 50  0001 C CNN
 	1    3500 2650
@@
 F 0 "CD600" H 5515 1596 50  0000 L CNN
 F 1 "0603 100nF" H 5515 1505 50  0000 L CNN
-F 2 "Samacsys:RESC1608X55N" H 5438 1400 50  0001 C CNN
+F 2 "" H 5438 1400 50  0001 C CNN
 F 3 "~" H 5400 1550 50  0001 C CNN
 	1    5400 1550
@@
 F 0 "CD602" H 7915 3546 50  0000 L CNN
 F 1 "0603 100nF" H 7915 3455 50  0000 L CNN
-F 2 "Samacsys:RESC1608X55N" H 7838 3350 50  0001 C CNN
+F 2 "" H 7838 3350 50  0001 C CNN
 F 3 "~" H 7800 3500 50  0001 C CNN
 	1    7800 3500
@@
 F 0 "CD604" H 9465 4546 50  0000 L CNN
 F 1 "0603 100nF" H 9465 4455 50  0000 L CNN
-F 2 "Samacsys:RESC1608X55N" H 9388 4350 50  0001 C CNN
+F 2 "" H 9388 4350 50  0001 C CNN
 F 3 "~" H 9350 4500 50  0001 C CNN
 	1    9350 4500
@@
 F 0 "U600" H 4250 5550 50  0000 L CNN
 F 1 "MK10DX128VLK7" H 4250 5450 50  0000 L CNN
-F 2 "Sparkdog PF-DI V2:MK10DX128VLK7" H 4250 5750 50  0001 C CNN
+F 2 "" H 4250 5750 50  0001 C CNN
 F 3 "" H 4250 5750 50  0001 C CNN
 	1    4250 5750
@@
 	4150 4050 3550 4050
 $Comp
-L Device:R_Pack04 RN606
+L Device:R_Pack04 RN605
 U 1 1 61FB3083
 P 3200 4450
-F 0 "RN606" V 2783 4450 50  0000 C CNN
+F 0 "RN605" V 2783 4450 50  0000 C CNN
 F 1 "1206 10k" V 2874 4450 50  0000 C CNN
-F 2 "Samacsys:742C083103JP" V 3475 4450 50  0001 C CNN
+F 2 "" V 3475 4450 50  0001 C CNN
 F 3 "~" H 3200 4450 50  0001 C CNN
 	1    3200 4450
@@
 Wire Wire Line
 	3400 4250 4150 4250
+Text Notes 7300 1050 0    50   ~ 0
+ETC PROCESSOR - can be used as an alternate low cost processor with Teensy not fitted.
 $EndSCHEMATC
