File: Sparkdog PF-DI V2/_autosave-Sparkdog PF-DI V2.sch (KiCad schematic (older format))
At the start: 12 parts, among them J1 Conn_01x06_Female, J2 Conn_01x08_Female, J3 Conn_01x06_Female, J4 Conn_01x08_Female, J5 Conn_01x06_Female, U2 Arduino_Footprint

Commit message: Commit schematic changes, new parts library footprints and step files, PCB design file.
Parts:
- J2, J4: footprint Sparkdog PF-DI V2:SIP-8 -> (none)
- J?: renamed from J1; footprint Sparkdog PF-DI V2:SIP-6 -> (none)
- J?: renamed from J3; footprint Sparkdog PF-DI V2:SIP-6 -> (none)
- J?: renamed from J5; footprint Sparkdog PF-DI V2:SIP-6 -> (none)
- RN100, RN101, RN102, RN103, RN104, RN105: footprint Samacsys:742C083103JP -> (none)
- U2: footprint Sparkdog PF-DI V2:ARDUINO_DUE -> (none)
Connections:
- net labels added: GDI1_SIG, GDI2_SIG
- net labels removed: GDI1_SIG_s, GDI2_SIG_s
Other:
- note removed: "SHEET 1 MASTER\nSHEET 2 VVT\nSHEET 3 TEENSY\nSHEET 4 KNOCK\nSHEET 5 ETC\nSHEET 6 ETC PROCESSOR\nSHEET 7 POWER\nSHEET 8 GDI\nSHEET 9 GDI CONTROL"
Changed lines of the file:
@@
 F 0 "U2" H 5750 5550 50  0000 C CNN
 F 1 "Arduino_Footprint" H 5500 5650 50  0000 C CNN
-F 2 "Sparkdog PF-DI V2:ARDUINO_DUE" H 5850 5500 50  0001 C CNN
+F 2 "" H 5850 5500 50  0001 C CNN
 F 3 "" H 5850 5500 50  0001 C CNN
 	1    5850 5500
@@
 ETC_O1B
 $Comp
-L Connector:Conn_01x06_Female J1
+L Connector:Conn_01x06_Female J?
 U 1 1 60E846D4
 P 2950 2000
-F 0 "J1" H 2978 1976 50  0000 L CNN
+F 0 "J?" H 2978 1976 50  0000 L CNN
 F 1 "Conn_01x06_Female" H 2500 2300 50  0000 L CNN
-F 2 "Sparkdog PF-DI V2:SIP-6" H 2950 2000 50  0001 C CNN
+F 2 "" H 2950 2000 50  0001 C CNN
 F 3 "~" H 2950 2000 50  0001 C CNN
 	1    2950 2000
@@
 $EndComp
 $Comp
-L Connector:Conn_01x06_Female J3
+L Connector:Conn_01x06_Female J?
 U 1 1 60E85A17
 P 2950 2700
-F 0 "J3" H 2978 2676 50  0000 L CNN
+F 0 "J?" H 2978 2676 50  0000 L CNN
 F 1 "Conn_01x06_Female" H 2500 3000 50  0000 L CNN
-F 2 "Sparkdog PF-DI V2:SIP-6" H 2950 2700 50  0001 C CNN
+F 2 "" H 2950 2700 50  0001 C CNN
 F 3 "~" H 2950 2700 50  0001 C CNN
 	1    2950 2700
@@
 $EndComp
 $Comp
-L Connector:Conn_01x06_Female J5
+L Connector:Conn_01x06_Female J?
 U 1 1 60E870A3
 P 2950 3400
-F 0 "J5" H 2978 3376 50  0000 L CNN
+F 0 "J?" H 2978 3376 50  0000 L CNN
 F 1 "Conn_01x06_Female" H 2500 3700 50  0000 L CNN
-F 2 "Sparkdog PF-DI V2:SIP-6" H 2950 3400 50  0001 C CNN
+F 2 "" H 2950 3400 50  0001 C CNN
 F 3 "~" H 2950 3400 50  0001 C CNN
 	1    2950 3400
@@
 PWIOD+
 Text Label 14800 5500 0    50   ~ 0
-GDI1_SIG_s
+GDI1_SIG
 Text Label 14800 5600 0    50   ~ 0
-GDI2_SIG_s
+GDI2_SIG
 Text Label 9400 8050 0    50   ~ 0
-GDI1_SIG_s
+GDI1_SIG
 Text Label 9400 8150 0    50   ~ 0
-GDI2_SIG_s
+GDI2_SIG
 Text Label 8200 8500 0    50   ~ 0
 ACH
@@
 F 0 "J2" H 2978 4176 50  0000 L CNN
 F 1 "Conn_01x08_Female" H 2500 4600 50  0000 L CNN
-F 2 "Sparkdog PF-DI V2:SIP-8" H 2950 4200 50  0001 C CNN
+F 2 "" H 2950 4200 50  0001 C CNN
 F 3 "~" H 2950 4200 50  0001 C CNN
 	1    2950 4200
@@
 F 0 "J4" H 3678 6376 50  0000 L CNN
 F 1 "Conn_01x08_Female" H 3200 6800 50  0000 L CNN
-F 2 "Sparkdog PF-DI V2:SIP-8" H 3650 6400 50  0001 C CNN
+F 2 "" H 3650 6400 50  0001 C CNN
 F 3 "~" H 3650 6400 50  0001 C CNN
 	1    3650 6400
@@
 F 0 "RN100" V 14083 5500 50  0000 C CNN
 F 1 "1206 10k" V 14174 5500 50  0000 C CNN
-F 2 "Samacsys:742C083103JP" V 14775 5500 50  0001 C CNN
+F 2 "" V 14775 5500 50  0001 C CNN
 F 3 "~" H 14500 5500 50  0001 C CNN
 	1    14500 5500
@@
 F 0 "RN101" V 6883 7900 50  0000 C CNN
 F 1 "1206 1k" V 6974 7900 50  0000 C CNN
-F 2 "Samacsys:742C083103JP" V 7575 7900 50  0001 C CNN
+F 2 "" V 7575 7900 50  0001 C CNN
 F 3 "~" H 7300 7900 50  0001 C CNN
 	1    7300 7900
@@
 F 0 "RN102" V 6883 9200 50  0000 C CNN
 F 1 "1206 1k" V 6974 9200 50  0000 C CNN
-F 2 "Samacsys:742C083103JP" V 7575 9200 50  0001 C CNN
+F 2 "" V 7575 9200 50  0001 C CNN
 F 3 "~" H 7300 9200 50  0001 C CNN
 	1    7300 9200
@@
 F 0 "RN103" V 9883 8250 50  0000 C CNN
 F 1 "1206 1k" V 9974 8250 50  0000 C CNN
-F 2 "Samacsys:742C083103JP" V 10575 8250 50  0001 C CNN
+F 2 "" V 10575 8250 50  0001 C CNN
 F 3 "~" H 10300 8250 50  0001 C CNN
 	1    10300 8250
@@
 F 0 "RN104" V 6883 9900 50  0000 C CNN
 F 1 "1206 10k" V 6974 9900 50  0000 C CNN
-F 2 "Samacsys:742C083103JP" V 7575 9900 50  0001 C CNN
+F 2 "" V 7575 9900 50  0001 C CNN
 F 3 "~" H 7300 9900 50  0001 C CNN
 	1    7300 9900
@@
 F 0 "RN105" V 9883 9100 50  0000 C CNN
 F 1 "1206 1k" V 9974 9100 50  0000 C CNN
-F 2 "Samacsys:742C083103JP" V 10575 9100 50  0001 C CNN
+F 2 "" V 10575 9100 50  0001 C CNN
 F 3 "~" H 10300 9100 50  0001 C CNN
 	1    10300 9100
@@
 Wire Wire Line
 	5600 3250 5750 3250
+Wire Bus Line
+	11050 8150 11050 10350
+Wire Bus Line
+	10150 4450 10450 4450
+Wire Bus Line
+	10700 1300 10700 2100
+Wire Bus Line
+	13900 1300 13900 6700
+Wire Bus Line
+	10150 3550 10550 3550
+Wire Bus Line
+	10550 2950 11100 2950
+Wire Bus Line
+	10650 2350 10650 4700
+Wire Bus Line
+	14650 1800 14650 3450
+Wire Bus Line
+	7000 6200 8100 6200
+Wire Bus Line
+	6350 6300 6350 10350
+Wire Bus Line
+	8100 7600 8100 8700
+Wire Bus Line
+	8100 6200 8100 7450
+Wire Bus Line
+	13700 1400 13700 5650
+Wire Bus Line
+	4600 1400 4600 4900
+Wire Bus Line
+	10650 4800 10650 6200
+Wire Bus Line
+	8100 6200 10650 6200
 Text GLabel 5600 3250 0    50   Output ~ 0
 VCC3V3
@@
 Text Notes 3900 3400 0    50   ~ 0
 5.0V RAIL INPUT FROM RABBIT ECU
-Text Notes 12650 9900 0    157  ~ 31
-SHEET 1 MASTER\nSHEET 2 VVT\nSHEET 3 TEENSY\nSHEET 4 KNOCK\nSHEET 5 ETC\nSHEET 6 ETC PROCESSOR\nSHEET 7 POWER\nSHEET 8 GDI\nSHEET 9 GDI CONTROL
-Wire Bus Line
-	11050 8150 11050 10350
-Wire Bus Line
-	10150 4450 10450 4450
-Wire Bus Line
-	10700 1300 10700 2100
-Wire Bus Line
-	13900 1300 13900 6700
-Wire Bus Line
-	10150 3550 10550 3550
-Wire Bus Line
-	10550 2950 11100 2950
-Wire Bus Line
-	10650 2350 10650 4700
-Wire Bus Line
-	14650 1800 14650 3450
-Wire Bus Line
-	7000 6200 8100 6200
-Wire Bus Line
-	6350 6300 6350 10350
-Wire Bus Line
-	8100 7600 8100 8700
-Wire Bus Line
-	8100 6200 8100 7450
-Wire Bus Line
-	13700 1400 13700 5650
-Wire Bus Line
-	4600 1400 4600 4900
-Wire Bus Line
-	10650 4800 10650 6200
-Wire Bus Line
-	8100 6200 10650 6200
 $EndSCHEMATC
