File: Sparkdog PF-DI V2/ETC PROCESSOR.sch (KiCad schematic (older format))
At the start: 21 parts, among them J600 M50-3610542R, U600 MK10DX128VLK7, U601 TLV809EA29DCKR, X600 Crystal

Commit message: Commit updates and Teensy schematic footprint correction.
Connections:
- net labels added: VCCA3V3
- net labels removed: VCC3V3A
Changed lines of the file:
@@
 	4150 5050 4100 5050
 Text GLabel 3500 5050 0    50   Input ~ 0
-VCC3V3A
+VCCA3V3
 Text GLabel 3500 5350 0    50   Input ~ 0
 VSSA

Commit message: Commit all files up to 21072021 Gerber and drill outputs.
Parts:
- added R601: 0603 1k, Samacsys:RESC1608X55N, symbol Device:R
Connections:
- net labels added: KTX
- wire segments 176 -> 179
Changed lines of the file:
@@
 	5450 5850 5450 7250
-Wire Wire Line
-	5650 5850 5650 7550
 Wire Wire Line
 	4250 7250 4250 7650
@@
 Text Notes 4000 6650 2    50   ~ 0
 DEBUG SWD PORT
-Text Label 5650 6600 1    50   ~ 0
+Text Label 5600 7550 2    50   ~ 0
 RESET
 Text Label 5450 6600 1    50   ~ 0
@@
 Wire Wire Line
 	3400 4250 4150 4250
+$Comp
+L Device:R R601
+U 1 1 60FD1D2F
+P 8000 4150
+F 0 "R601" V 8207 4150 50  0000 C CNN
+F 1 "0603 1k" V 8116 4150 50  0000 C CNN
+F 2 "Samacsys:RESC1608X55N" V 7930 4150 50  0001 C CNN
+F 3 "~" H 8000 4150 50  0001 C CNN
+	1    8000 4150
+	0    -1   -1   0
+$EndComp
+Wire Wire Line
+	7050 4350 7700 4350
+Wire Wire Line
+	7700 4350 7700 4150
+Wire Wire Line
+	7700 4150 7850 4150
+Wire Wire Line
+	8150 4150 8500 4150
+Text HLabel 8500 4150 2    50   Input ~ 0
+KTX
+Text Label 7750 5250 0    50   ~ 0
+RESET
 $EndSCHEMATC
