File: Sparkdog PF-DI V2/ETC.sch (KiCad schematic (older format))
At the start: 37 parts, among them U500 L6206PD013TR, U501 SUD19P06-60, U502 TL331SN4T3G, U503 Dual_Trans_Array_NPN

Commit message: Commit schematic changes, new parts library footprints and step files, PCB design file.
Parts:
- C500, C501, C502, C503, C504, CD501, CD502, R500, R501, R502, R503, R506, R511, R512, R513, R514, R515: footprint (none) -> Samacsys:RESC1608X55N
- C505, C506, D500, D501, D502, D503, D504, R507, R508, R509, R510: footprint (none) -> Samacsys:RESC2012X60N
- CD500: value 2mm 4.7uF -> CAP4mm 4.7uF; footprint (none) -> Samacsys:CAPAE1700X1700N
- R504, R505: value 1206 0.1R -> 2512 0.1R; footprint (none) -> Samacsys:RESC6331X75N
- RN500, RN501: footprint (none) -> Samacsys:742C083103JP
- U500: footprint SOP65P1420X360-37N -> Samacsys:SOP65P1420X360-37N
- U501: footprint Package_TO_SOT_SMD:TO-252-2 -> Sparkdog PF-DI V2:MDAC-TO-252-3
- U502: footprint SOT95P275X110-5N -> Samacsys:SOT95P275X110-5N
- U503: footprint (none) -> Sparkdog PF-DI V2:SOT-363-6
Connections:
- net labels added: ETC_ENA_s, ETC_ENB_s, ETC_IFA_s, ETC_IFB_s, ETC_IN1A_s, ETC_IN1B_s, ETC_IN2A_s, ETC_IN2B_s, ETC_O1A_s, ETC_O1B_s, ETC_O2A_s, ETC_O2B_s, ETC_VFB_s, ETC_VFF_s

Commit message: Commit all files up to 21072021 Gerber and drill outputs.
Connections:
- net labels added: VCC12VPP
- net labels removed: VCC12VP
Changed lines of the file:
@@
 	4400 2650 5500 2650
 Text GLabel 5600 2650 2    50   Input ~ 0
-VCC12VP
+VCC12VPP
 $Comp
 L Device:R R511
