File: Sparkdog PF-DI V2/GDI.sch (KiCad schematic (older format))
At the start: 54 parts, among them U800 DDC113TU, U801 DDC113TU, U802 DDC113TU, U803 STD7NK40Z, U804 STD7NK40Z, U805 SUD19P06-60, U806 SUD19P06-60, U807 SUD19P06-60, U808 SUD19P06-60, U809 Dual_Trans_Array_NPN, U810 STD7NK40Z, U811 STD7NK40Z, U850 DDC113TU, U851 DDC113TU, U852 DDC113TU, U853 STD7NK40Z, U854 STD7NK40Z, U855 SUD19P06-60, U856 SUD19P06-60, U857 SUD19P06-60, U858 SUD19P06-60

Commit message: Commit schematic changes, new parts library footprints and step files, PCB design file.
Parts:
- D800, D801, D802, D803, D850, D851, D852, D853: footprint (none) -> Samacsys:DIOM5127X229N
- D804: value D_Zener -> DO-214AC 81V; footprint (none) -> Samacsys:DIOM5127X229N
- D805: value SCHOTTKY -> DO-214AC SCHOTTKY; footprint (none) -> Samacsys:DIOM5127X229N
- R800, R803, R804, R805, R806, R807, R808, R809, R811, R812, R850, R853, R854, R855, R856, R857, R858, R859: footprint (none) -> Samacsys:RESC1608X55N
- R801, R851: value 1210 4.7k -> 1206 4.7k; footprint (none) -> Samacsys:RESC3216X60N
- R802, R852: footprint (none) -> Samacsys:RESC6331X75N
- R810: value 1206 0.2R -> 2512 0.2R; footprint (none) -> Samacsys:RESC6331X75N
- U800, U801, U802, U809, U850, U851, U852: footprint (none) -> Sparkdog PF-DI V2:SOT-363-6
- U803, U804, U805, U806, U807, U808, U810, U811, U853, U854, U855, U856, U857, U858: footprint Package_TO_SOT_SMD:TO-252-2 -> Sparkdog PF-DI V2:MDAC-TO-252-3
Connections:
- net labels added: SIG_PWM_LSAB_s, SIG_PWM_LSCD_s

Commit message: Commit all files up to 21072021 Gerber and drill outputs.
Connections:
- net labels added: VCC12VPP
- net labels removed: VCC12V, VCC12VP
Changed lines of the file:
@@
 Connection ~ 10200 1400
 Text GLabel 10250 1400 2    50   Input ~ 0
-VCC12V
+VCC12VPP
 Text GLabel 9650 2300 2    50   Input ~ 0
 VCC50VPP
@@
 Connection ~ 7700 1400
 Text GLabel 7750 1400 2    50   Input ~ 0
-VCC12V
+VCC12VPP
 Text GLabel 7150 2300 2    50   Input ~ 0
 VCC50VPP
@@
 Connection ~ 10200 3750
 Text GLabel 10250 3750 2    50   Input ~ 0
-VCC12V
+VCC12VPP
 Text GLabel 9650 4650 2    50   Input ~ 0
 VCC50VPP
@@
 Connection ~ 7700 3750
 Text GLabel 7750 3750 2    50   Input ~ 0
-VCC12V
+VCC12VPP
 Text GLabel 7150 4650 2    50   Input ~ 0
 VCC50VPP
@@
 	5750 1900 5800 1900
 Text GLabel 5500 2500 2    50   Input ~ 0
-VCC12V
+VCC12VPP
 $Comp
 L Device:R R802
@@
 	5750 4250 5800 4250
 Text GLabel 5500 4850 2    50   Input ~ 0
-VCC12V
+VCC12VPP
 $Comp
 L Device:R R852
@@
 	6250 7350 6350 7350
 Text GLabel 6350 7350 2    50   Input ~ 0
-VCC12VP
+VCC12VPP
 $Comp
 L Device:D_Schottky D805
