File: Sparkdog PF-DI V2/Power.sch (KiCad schematic (older format))
At the start: 36 parts, among them J700 SSM-106-L-SV, U700 BD433M5FP-CE2, U701 PIC18F26J50T-I_ML, U702 TCAN334, U703 BD433M5FP-CE2, U704 LM2577SX-ADJ_NOPB, X700 4 MHz

Commit message: Commit schematic changes, new parts library footprints and step files, PCB design file.
Parts:
- C700, C701, C702, CD705, CD706, CD708, CD712, CD714, R700, R701, R702, R703, R705, R706: footprint (none) -> Samacsys:RESC1608X55N
- CD700, CD701, CD703: value 100nF -> 0603 100nF; footprint (none) -> Samacsys:RESC1608X55N
- CD702, CD704: value 4.7uF -> CAP4mm 4.7uF; footprint (none) -> Samacsys:CAPAE430X550N
- CD707, CD711: value CP -> CAP4mm 4.7uF; footprint (none) -> Samacsys:CAPAE430X550N
- CD709: value CP -> CAP17mm; footprint (none) -> Samacsys:CAPAE1700X1700N
- CD710: value 0805 100nF -> 0603 100nF; footprint (none) -> Samacsys:RESC1608X55N
- CD713: value C -> 0603 100nF; footprint (none) -> Samacsys:RESC1608X55N
- D700: footprint (none) -> Samacsys:DIOM5127X229N
- J700: footprint SSM106LSV -> Samacsys:SSM106LSV
- L700, L701: value L -> 0805 10nH; footprint (none) -> Samacsys:RESC2012X60N
- L702: footprint (none) -> Samacsys:INDC8566X410N
- R704: footprint (none) -> Samacsys:RESC6331X75N
- U700, U703: footprint BD433M5FPCE2 -> Sparkdog PF-DI V2:MDAC-TO-252-3
- U701: footprint QFN65P600X600X100-29N-D -> Sparkdog PF-DI V2:PIC18F26
- U702: footprint (none) -> Samacsys:SOIC127P600X175-8N
- U704: footprint KTT0005B -> Samacsys:KTT0005B
- X700: footprint (none) -> Samacsys:ECS49205PXTR
Changed lines of the file:
@@
 P 2850 1400
 F 0 "CD700" H 2965 1446 50  0000 L CNN
-F 1 "100nF" H 2965 1355 50  0000 L CNN
-F 2 "" H 2888 1250 50  0001 C CNN
+F 1 "0603 100nF" H 2965 1355 50  0000 L CNN
+F 2 "Samacsys:RESC1608X55N" H 2888 1250 50  0001 C CNN
 F 3 "~" H 2850 1400 50  0001 C CNN
 	1    2850 1400
@@
 P 2850 1900
 F 0 "CD701" H 2965 1946 50  0000 L CNN
-F 1 "100nF" H 2965 1855 50  0000 L CNN
-F 2 "" H 2888 1750 50  0001 C CNN
+F 1 "0603 100nF" H 2965 1855 50  0000 L CNN
+F 2 "Samacsys:RESC1608X55N" H 2888 1750 50  0001 C CNN
 F 3 "~" H 2850 1900 50  0001 C CNN
 	1    2850 1900
@@
 P 3350 1900
 F 0 "CD703" H 3465 1946 50  0000 L CNN
-F 1 "100nF" H 3465 1855 50  0000 L CNN
-F 2 "" H 3388 1750 50  0001 C CNN
+F 1 "0603 100nF" H 3465 1855 50  0000 L CNN
+F 2 "Samacsys:RESC1608X55N" H 3388 1750 50  0001 C CNN
 F 3 "~" H 3350 1900 50  0001 C CNN
 	1    3350 1900
@@
 P 3350 1400
 F 0 "CD702" H 3468 1446 50  0000 L CNN
-F 1 "4.7uF" H 3468 1355 50  0000 L CNN
-F 2 "" H 3388 1250 50  0001 C CNN
+F 1 "CAP4mm 4.7uF" H 3468 1355 50  0000 L CNN
+F 2 "Samacsys:CAPAE430X550N" H 3388 1250 50  0001 C CNN
 F 3 "~" H 3350 1400 50  0001 C CNN
 	1    3350 1400
@@
 P 4150 1900
 F 0 "CD704" H 4033 1854 50  0000 R CNN
-F 1 "4.7uF" H 4033 1945 50  0000 R CNN
-F 2 "" H 4188 1750 50  0001 C CNN
+F 1 "CAP4mm 4.7uF" H 4033 1945 50  0000 R CNN
+F 2 "Samacsys:CAPAE430X550N" H 4188 1750 50  0001 C CNN
 F 3 "~" H 4150 1900 50  0001 C CNN
 	1    4150 1900
@@
 P 4500 1650
 F 0 "L700" V 4319 1650 50  0000 C CNN
-F 1 "L" V 4410 1650 50  0000 C CNN
-F 2 "" H 4500 1650 50  0001 C CNN
+F 1 "0805 10nH" V 4410 1650 50  0000 C CNN
+F 2 "Samacsys:RESC2012X60N" H 4500 1650 50  0001 C CNN
 F 3 "~" H 4500 1650 50  0001 C CNN
 	1    4500 1650
@@
 P 4500 2100
 F 0 "L701" V 4319 2100 50  0000 C CNN
-F 1 "L" V 4410 2100 50  0000 C CNN
-F 2 "" H 4500 2100 50  0001 C CNN
+F 1 "0805 10nH" V 4410 2100 50  0000 C CNN
+F 2 "Samacsys:RESC2012X60N" H 4500 2100 50  0001 C CNN
 F 3 "~" H 4500 2100 50  0001 C CNN
 	1    4500 2100
@@
 F 0 "CD705" H 4915 1896 50  0000 L CNN
 F 1 "0603 100nF" H 4915 1805 50  0000 L CNN
-F 2 "" H 4838 1700 50  0001 C CNN
+F 2 "Samacsys:RESC1608X55N" H 4838 1700 50  0001 C CNN
 F 3 "~" H 4800 1850 50  0001 C CNN
 	1    4800 1850
@@
 F 0 "U704" H 7850 1865 50  0000 C CNN
 F 1 "LM2577SX-ADJ_NOPB" H 7850 1774 50  0000 C CNN
-F 2 "KTT0005B" H 8400 1700 50  0001 L CNN
+F 2 "Samacsys:KTT0005B" H 8400 1700 50  0001 L CNN
 F 3 "http://www.ti.com/lit/gpn/LM2577" H 8400 1600 50  0001 L CNN
 F 4 "SIMPLE SWITCHER&#174; 3.5V to 40V, 3A Low Component Count Step-Up Regulator" H 8400 1500 50  0001 L CNN "Description"
@@
 F 0 "R702" V 7300 2000 50  0000 C CNN
 F 1 "0603 22k" V 7200 2000 50  0000 C CNN
-F 2 "" V 7030 2100 50  0001 C CNN
+F 2 "Samacsys:RESC1608X55N" V 7030 2100 50  0001 C CNN
 F 3 "~" H 7100 2100 50  0001 C CNN
 	1    7100 2100
@@
 P 9250 1850
 F 0 "CD710" H 9365 1896 50  0000 L CNN
-F 1 "0805 100nF" H 9365 1805 50  0000 L CNN
-F 2 "" H 9288 1700 50  0001 C CNN
+F 1 "0603 100nF" H 9365 1805 50  0000 L CNN
+F 2 "Samacsys:RESC1608X55N" H 9288 1700 50  0001 C CNN
 F 3 "~" H 9250 1850 50  0001 C CNN
 	1    9250 1850
@@
 P 10150 1850
 F 0 "CD711" H 10268 1896 50  0000 L CNN
-F 1 "CP" H 10268 1805 50  0000 L CNN
-F 2 "" H 10188 1700 50  0001 C CNN
+F 1 "CAP4mm 4.7uF" H 10268 1805 50  0000 L CNN
+F 2 "Samacsys:CAPAE430X550N" H 10188 1700 50  0001 C CNN
 F 3 "~" H 10150 1850 50  0001 C CNN
 	1    10150 1850
@@
 F 0 "L702" V 9600 1400 50  0000 C CNN
 F 1 "SRN8040-680" V 9700 1650 50  0000 C CNN
-F 2 "" H 9000 1600 50  0001 C CNN
+F 2 "Samacsys:INDC8566X410N" H 9000 1600 50  0001 C CNN
 F 3 "~" H 9000 1600 50  0001 C CNN
 	1    9000 1600
@@
 F 0 "D700" H 9000 1233 50  0000 C CNN
 F 1 "BYG22B" H 9000 1324 50  0000 C CNN
-F 2 "" H 9000 1450 50  0001 C CNN
+F 2 "Samacsys:DIOM5127X229N" H 9000 1450 50  0001 C CNN
 F 3 "~" H 9000 1450 50  0001 C CNN
 	1    9000 1450
@@
 P 9400 1300
 F 0 "CD709" H 9282 1254 50  0000 R CNN
-F 1 "CP" H 9282 1345 50  0000 R CNN
-F 2 "" H 9438 1150 50  0001 C CNN
+F 1 "CAP17mm" H 9282 1345 50  0000 R CNN
+F 2 "Samacsys:CAPAE1700X1700N" H 9438 1150 50  0001 C CNN
 F 3 "~" H 9400 1300 50  0001 C CNN
 	1    9400 1300
@@
 F 0 "R701" V 6807 2100 50  0000 C CNN
 F 1 "0603 1k" V 6716 2100 50  0000 C CNN
-F 2 "" V 6530 2100 50  0001 C CNN
+F 2 "Samacsys:RESC1608X55N" V 6530 2100 50  0001 C CNN
 F 3 "~" H 6600 2100 50  0001 C CNN
 	1    6600 2100
@@
 F 0 "R700" V 6793 1600 50  0000 C CNN
 F 1 "0603 1k" V 6884 1600 50  0000 C CNN
-F 2 "" V 6930 1600 50  0001 C CNN
+F 2 "Samacsys:RESC1608X55N" V 6930 1600 50  0001 C CNN
 F 3 "~" H 7000 1600 50  0001 C CNN
 	1    7000 1600
@@
 F 0 "C700" V 6398 1600 50  0000 C CNN
 F 1 "0603 100nF" V 6489 1600 50  0000 C CNN
-F 2 "" H 6688 1450 50  0001 C CNN
+F 2 "Samacsys:RESC1608X55N" H 6688 1450 50  0001 C CNN
 F 3 "~" H 6650 1600 50  0001 C CNN
 	1    6650 1600
@@
 F 0 "R703" V 7750 2050 50  0000 C CNN
 F 1 "0603 22k" V 7650 2050 50  0000 C CNN
-F 2 "" V 7480 2100 50  0001 C CNN
+F 2 "Samacsys:RESC1608X55N" V 7480 2100 50  0001 C CNN
 F 3 "~" H 7550 2100 50  0001 C CNN
 	1    7550 2100
@@
 F 0 "U701" H 2250 6850 50  0000 L CNN
 F 1 "PIC18F26J50T-I_ML" H 2250 6750 50  0000 L CNN
-F 2 "QFN65P600X600X100-29N-D" H 5600 6500 50  0001 L CNN
+F 2 "Sparkdog PF-DI V2:PIC18F26" H 5600 6500 50  0001 L CNN
 F 3 "https://componentsearchengine.com/Datasheets/1/PIC18F26J50T-I_ML.pdf" H 5600 6400 50  0001 L CNN
 F 4 "8-bit Microcontrollers - MCU Full Spd USB 64KB Flsh 4KBRAM nanoWatt" H 5600 6300 50  0001 L CNN "Description"
@@
 F 0 "U700" H 1950 1915 50  0000 C CNN
 F 1 "BD433M5FP-CE2" H 1950 1824 50  0000 C CNN
-F 2 "BD433M5FPCE2" H 2350 1750 50  0001 L CNN
+F 2 "Sparkdog PF-DI V2:MDAC-TO-252-3" H 2350 1750 50  0001 L CNN
 F 3 "" H 2350 1650 50  0001 L CNN
 F 4 "ROHM - BD433M5FP-CE2 - LDO, FIXED, AUTO, 3.3V, 0.5A, TO252-3" H 2350 1550 50  0001 L CNN "Description"
@@
 F 0 "U703" H 9150 4915 50  0000 C CNN
 F 1 "BD433M5FP-CE2" H 9150 4824 50  0000 C CNN
-F 2 "BD433M5FPCE2" H 9550 4750 50  0001 L CNN
+F 2 "Sparkdog PF-DI V2:MDAC-TO-252-3" H 9550 4750 50  0001 L CNN
 F 3 "" H 9550 4650 50  0001 L CNN
 F 4 "ROHM - BD433M5FP-CE2 - LDO, FIXED, AUTO, 3.3V, 0.5A, TO252-3" H 9550 4550 50  0001 L CNN "Description"
@@
 F 0 "CD712" H 7165 4546 50  0000 L CNN
 F 1 "0603 100nF" H 7165 4455 50  0000 L CNN
-F 2 "" H 7088 4350 50  0001 C CNN
+F 2 "Samacsys:RESC1608X55N" H 7088 4350 50  0001 C CNN
 F 3 "~" H 7050 4500 50  0001 C CNN
 	1    7050 4500
@@
 F 0 "CD708" H 7765 4946 50  0000 L CNN
 F 1 "0603 100nF" H 7765 4855 50  0000 L CNN
-F 2 "" H 7688 4750 50  0001 C CNN
+F 2 "Samacsys:RESC1608X55N" H 7688 4750 50  0001 C CNN
 F 3 "~" H 7650 4900 50  0001 C CNN
 	1    7650 4900
@@
 P 7100 4900
 F 0 "CD707" H 7218 4946 50  0000 L CNN
-F 1 "CP" H 7218 4855 50  0000 L CNN
-F 2 "" H 7138 4750 50  0001 C CNN
+F 1 "CAP4mm 4.7uF" H 7218 4855 50  0000 L CNN
+F 2 "Samacsys:CAPAE430X550N" H 7138 4750 50  0001 C CNN
 F 3 "~" H 7100 4900 50  0001 C CNN
 	1    7100 4900
@@
 F 0 "CD706" H 6465 5696 50  0000 L CNN
 F 1 "0603 100nF" H 6465 5605 50  0000 L CNN
-F 2 "" H 6388 5500 50  0001 C CNN
+F 2 "Samacsys:RESC1608X55N" H 6388 5500 50  0001 C CNN
 F 3 "~" H 6350 5650 50  0001 C CNN
 	1    6350 5650
@@
 F 0 "U702" H 6750 3950 50  0000 C CNN
 F 1 "TCAN334" H 6800 3850 50  0000 C CNN
-F 2 "" H 7450 2950 50  0001 C CIN
+F 2 "Samacsys:SOIC127P600X175-8N" H 7450 2950 50  0001 C CIN
 F 3 "http://www.ti.com/lit/ds/symlink/tcan337.pdf" H 7450 3450 50  0001 C CNN
 	1    7450 3450
@@
 P 7800 2900
 F 0 "CD713" H 7915 2946 50  0000 L CNN
-F 1 "C" H 7915 2855 50  0000 L CNN
-F 2 "" H 7838 2750 50  0001 C CNN
+F 1 "0603 100nF" H 7915 2855 50  0000 L CNN
+F 2 "Samacsys:RESC1608X55N" H 7838 2750 50  0001 C CNN
 F 3 "~" H 7800 2900 50  0001 C CNN
 	1    7800 2900
@@
 F 0 "R704" H 10220 1346 50  0000 L CNN
 F 1 "2512 1R" H 10220 1255 50  0000 L CNN
-F 2 "" V 10080 1300 50  0001 C CNN
+F 2 "Samacsys:RESC6331X75N" V 10080 1300 50  0001 C CNN
 F 3 "~" H 10150 1300 50  0001 C CNN
 	1    10150 1300
@@
 F 0 "R706" V 4493 2600 50  0000 C CNN
 F 1 "0603 1k" V 4584 2600 50  0000 C CNN
-F 2 "" V 4630 2600 50  0001 C CNN
+F 2 "Samacsys:RESC1608X55N" V 4630 2600 50  0001 C CNN
 F 3 "~" H 4700 2600 50  0001 C CNN
 	1    4700 2600
@@
 F 0 "CD714" H 1415 5496 50  0000 L CNN
 F 1 "0603 100nF" H 1415 5405 50  0000 L CNN
-F 2 "" H 1338 5300 50  0001 C CNN
+F 2 "Samacsys:RESC1608X55N" H 1338 5300 50  0001 C CNN
 F 3 "~" H 1300 5450 50  0001 C CNN
 	1    1300 5450
@@
 F 0 "X700" H 2100 6368 50  0000 C CNN
 F 1 "4 MHz" H 2100 6277 50  0000 C CNN
-F 2 "" H 2100 6100 50  0001 C CNN
+F 2 "Samacsys:ECS49205PXTR" H 2100 6100 50  0001 C CNN
 F 3 "~" H 2100 6100 50  0001 C CNN
 	1    2100 6100
@@
 F 0 "C702" H 1400 6600 50  0000 L CNN
 F 1 "0603 10pF" H 1400 6500 50  0000 L CNN
-F 2 "" H 2288 6350 50  0001 C CNN
+F 2 "Samacsys:RESC1608X55N" H 2288 6350 50  0001 C CNN
 F 3 "~" H 2250 6500 50  0001 C CNN
 	1    2250 6500
@@
 F 0 "C701" H 900 6600 50  0000 L CNN
 F 1 "0603 10pF" H 900 6500 50  0000 L CNN
-F 2 "" H 1988 6350 50  0001 C CNN
+F 2 "Samacsys:RESC1608X55N" H 1988 6350 50  0001 C CNN
 F 3 "~" H 1950 6500 50  0001 C CNN
 	1    1950 6500
@@
 F 0 "J700" V 2300 1650 50  0000 L CNN
 F 1 "SSM-106-L-SV" V 2400 1650 50  0000 L CNN
-F 2 "SSM106LSV" H 2550 2700 50  0001 L CNN
+F 2 "Samacsys:SSM106LSV" H 2550 2700 50  0001 L CNN
 F 3 "http://suddendocs.samtec.com/catalog_english/ssm_sm.pdf" H 2550 2600 50  0001 L CNN
 F 4 "Samtec SSM Series 2.54mm 6 Way 1 Row Straight PCB Socket Surface Mount Board to Board" H 2550 2500 50  0001 L CNN "Description"
@@
 F 0 "R705" V 1043 5200 50  0000 C CNN
 F 1 "0603 100k" V 1134 5200 50  0000 C CNN
-F 2 "" V 1180 5200 50  0001 C CNN
+F 2 "Samacsys:RESC1608X55N" V 1180 5200 50  0001 C CNN
 F 3 "~" H 1250 5200 50  0001 C CNN
 	1    1250 5200
@@
 Wire Wire Line
 	1400 5200 2350 5200
+Text GLabel 3650 3500 1    50   Input ~ 0
+VSS
 $EndSCHEMATC

Commit message: Commit all files up to 21072021 Gerber and drill outputs.
Connections:
- net labels added: ANK1, ANK2, KTX, VCC12VPP
- wire segments 122 -> 128
Changed lines of the file:
@@
 	9400 1700 10150 1700
 Text GLabel 10350 1700 2    50   Input ~ 0
-VCC12VP
+VCC12VPP
 Wire Wire Line
 	10350 2000 10150 2000
@@
 Text GLabel 3650 3500 1    50   Input ~ 0
 VSS
+Wire Wire Line
+	3950 7100 3950 7450
+Wire Wire Line
+	3950 7450 3500 7450
+Text HLabel 3500 7450 0    50   Input ~ 0
+ANK1
+Text HLabel 3700 2950 0    50   Input ~ 0
+ANK2
+Wire Wire Line
+	3750 3500 3750 2950
+Wire Wire Line
+	3750 2950 3700 2950
+Wire Wire Line
+	4350 7100 4350 7550
+Wire Wire Line
+	4350 7550 3500 7550
+Text HLabel 3500 7550 0    50   Input ~ 0
+KTX
 $EndSCHEMATC
