File: Sparkdog PF-DI V2/Sparkdog PF-DI V2.sch (KiCad schematic (older format))
At the start: 12 parts, among them J1 Conn_01x06_Female, J2 Conn_01x08_Female, J3 Conn_01x06_Female, J4 Conn_01x08_Female, J5 Conn_01x06_Female, U2 Arduino_Footprint

Commit message: Commit running changes for safekeeping
Changed lines of the file:
@@
 Wire Wire Line
 	3100 6600 3450 6600
-Text GLabel 3450 6100 0    50   Input ~ 0
-VSS
-Text GLabel 3450 6200 0    50   Input ~ 0
-VSS
-Text GLabel 3450 6300 0    50   Input ~ 0
-VSS
-Text GLabel 3450 6400 0    50   Input ~ 0
-VSS
-Text GLabel 3450 6500 0    50   Input ~ 0
-VSS
 Wire Wire Line
 	9950 4150 10250 4150

Commit message: Commit for safekeeping
Connections:
- wire segments 284 -> 287
Changed lines of the file:
@@
 Text Notes 12650 9900 0    157  ~ 31
 SHEET 1 MASTER\nSHEET 2 VVT\nSHEET 3 TEENSY\nSHEET 4 KNOCK\nSHEET 5 ETC\nSHEET 6 ETC PROCESSOR\nSHEET 7 POWER\nSHEET 8 GDI\nSHEET 9 GDI CONTROL
+Text GLabel 6100 5700 0    50   Input ~ 0
+VSS
+Wire Wire Line
+	6100 5550 6100 5700
+Wire Wire Line
+	6200 5700 6200 5550
+Wire Wire Line
+	6200 5700 6100 5700
 Wire Bus Line
 	11050 8150 11050 10350

Commit message: Commit all files up to 21072021 Gerber and drill outputs.
Parts:
- added C100: 0603 100nF, Samacsys:RESC1608X55N, symbol Device:C
- added R100, R101: 0603 1k, Samacsys:RESC1608X55N, symbol Device:R
- added RN106: 1206 10k, Samacsys:742C083103JP, symbol Device:R_Pack04
Connections:
- net labels added: SIG_KTX, VCC12VPP
- net labels removed: VCC12
- wire segments 287 -> 315
Other:
- note added: "RC PWM to VOLT converter when T3.5 not used"
Changed lines of the file:
@@
 MISO
 $Sheet
-S 2450 6450 650  550
+S 2450 6450 650  1050
 U 60642A2F
 F0 "7 POWER" 50
@@
 F4 "SIG_CANL" I R 3100 6700 50
 F5 "SIG_KRQ" I R 3100 6900 50
+F6 "ANK1" I R 3100 7100 50
+F7 "ANK2" I R 3100 7200 50
+F8 "KTX" I R 3100 7300 50
 $EndSheet
 $Sheet
@@
 	10300 7450 9950 7450
 Text Label 10000 7450 0    50   ~ 0
+PPSM
+Text Label 10000 7550 0    50   ~ 0
 TPSM
-Text Label 10000 7550 0    50   ~ 0
-TPSS
 Wire Wire Line
 	9950 7550 10300 7550
@@
 VSS
 Text GLabel 2350 1900 0    50   Input ~ 0
-VCC12
+VCC12VPP
 Text Label 2400 2000 0    50   ~ 0
 PWIOAB-
@@
 SIG_K2IN
 Text Label 12250 7150 0    50   ~ 0
-SIG_K2IN
+SIG_K1IN
 Text GLabel 2750 4000 0    50   Input ~ 0
 VSS
@@
 Wire Wire Line
 	14700 5600 15300 5600
-Wire Wire Line
-	5300 5050 5750 5050
 Wire Wire Line
 	6300 5550 6300 6100
@@
 	7300 5550 7300 6100
 $Sheet
-S 8550 6750 750  3100
+S 8550 6750 750  3250
 U 60717C73
 F0 "6 ETC PROCESSOR" 50
@@
 F52 "SIG_DM2" I L 8550 8800 50
 F53 "SIG_DP2" I L 8550 8700 50
+F54 "KTX" I L 8550 9800 50
 $EndSheet
 Wire Wire Line
@@
 Wire Wire Line
 	6200 5700 6100 5700
+Entry Wire Line
+	8000 6550 8100 6650
+Wire Wire Line
+	8000 6550 7600 6550
+Text Label 7650 6550 0    50   ~ 0
+REL_RST
+$Comp
+L Device:R R100
+U 1 1 60F627BD
+P 7450 6550
+F 0 "R100" V 7243 6550 50  0000 C CNN
+F 1 "0603 1k" V 7334 6550 50  0000 C CNN
+F 2 "Samacsys:RESC1608X55N" V 7380 6550 50  0001 C CNN
+F 3 "~" H 7450 6550 50  0001 C CNN
+	1    7450 6550
+	0    1    1    0
+$EndComp
+Wire Wire Line
+	7100 6550 7300 6550
+Text GLabel 7100 6550 0    50   Input ~ 0
+VCC3V3
+Wire Wire Line
+	9500 5550 9500 5650
+Wire Wire Line
+	9500 5650 9600 5650
+Wire Wire Line
+	9600 5650 9600 5550
+Wire Wire Line
+	9600 5650 9650 5650
+Connection ~ 9600 5650
+Text GLabel 9650 5650 2    50   Input ~ 0
+VCC5V
+Wire Wire Line
+	3100 7100 3650 7100
+Wire Wire Line
+	3100 7200 3650 7200
+Wire Wire Line
+	3100 7300 3650 7300
+Text Label 3300 7100 0    50   ~ 0
+SIG_K1O
+Text Label 3300 7200 0    50   ~ 0
+SIG_K2O
+Text Label 3300 7300 0    50   ~ 0
+SIG_KTX
+Wire Wire Line
+	8550 9800 8150 9800
+Text Label 8200 9800 0    50   ~ 0
+SIG_KTX
+$Comp
+L Device:R_Pack04 RN106
+U 1 1 6101B7F5
+P 5100 6850
+F 0 "RN106" V 4683 6850 50  0000 C CNN
+F 1 "1206 10k" V 4774 6850 50  0000 C CNN
+F 2 "Samacsys:742C083103JP" V 5375 6850 50  0001 C CNN
+F 3 "~" H 5100 6850 50  0001 C CNN
+	1    5100 6850
+	0    1    1    0
+$EndComp
+Wire Wire Line
+	5300 6950 6000 6950
+Text Label 5400 6950 0    50   ~ 0
+SIG_VVTB_OUT
+$Comp
+L Device:C C100
+U 1 1 6106D199
+P 4300 6500
+F 0 "C100" H 4415 6546 50  0000 L CNN
+F 1 "0603 100nF" H 4415 6455 50  0000 L CNN
+F 2 "Samacsys:RESC1608X55N" H 4338 6350 50  0001 C CNN
+F 3 "~" H 4300 6500 50  0001 C CNN
+	1    4300 6500
+	1    0    0    -1
+$EndComp
+Wire Wire Line
+	4300 6650 4900 6650
+Text GLabel 4300 6350 0    50   Input ~ 0
+VSS
+Text Notes 4200 7150 0    50   ~ 0
+RC PWM to VOLT converter when T3.5 not used
+Wire Wire Line
+	5100 5050 5100 6200
+Wire Wire Line
+	5100 6200 5500 6200
+Wire Wire Line
+	5500 6200 5500 6650
+Wire Wire Line
+	5500 6650 5300 6650
+Wire Wire Line
+	5100 5050 5750 5050
+Wire Wire Line
+	4900 6950 4900 6850
+Wire Wire Line
+	5300 6850 5300 6750
+Wire Wire Line
+	4900 6750 4900 6650
+Connection ~ 4900 6650
+Entry Wire Line
+	6650 6100 6750 6200
+Wire Wire Line
+	6650 6100 6650 5800
+Wire Wire Line
+	6650 5800 4800 5800
+Text Label 6650 6050 1    50   ~ 0
+HMEN
+$Comp
+L Device:R R101
+U 1 1 611BAC47
+P 4650 5800
+F 0 "R101" V 4443 5800 50  0000 C CNN
+F 1 "0603 1k" V 4534 5800 50  0000 C CNN
+F 2 "Samacsys:RESC1608X55N" V 4580 5800 50  0001 C CNN
+F 3 "~" H 4650 5800 50  0001 C CNN
+	1    4650 5800
+	0    1    1    0
+$EndComp
+Wire Wire Line
+	4500 5800 4150 5800
+Text Label 4200 5800 0    50   ~ 0
+ETC_1A
+Text Notes 4250 5950 0    50   ~ 0
+OVERRIDE NO T3.5
+Wire Wire Line
+	3950 9450 3850 9450
+Wire Wire Line
+	3850 9450 3850 10000
+Wire Wire Line
+	3850 10000 3200 10000
+Wire Wire Line
+	3200 9900 3750 9900
+Wire Wire Line
+	3750 9900 3750 9350
+Wire Wire Line
+	3750 9350 3950 9350
+Text Label 3250 9900 0    50   ~ 0
+GDI1_SIG_s
 Wire Bus Line
 	11050 8150 11050 10350
@@
 	14650 1800 14650 3450
 Wire Bus Line
-	7000 6200 8100 6200
+	6750 6200 8100 6200
 Wire Bus Line
 	6350 6300 6350 10350
@@
 Wire Bus Line
 	8100 6200 10650 6200
+Text Label 3250 10000 0    50   ~ 0
+GDI2_SIG_s
 $EndSCHEMATC
